File: pnp/pcb/mobo/mosfets.kicad_sch (KiCad schematic)
At the start: 0 parts

Commit message: Redesign finished
Completed Board redesign and adding more EMC improvements.
Changed all the part numbers to have a Mouser orderable design (except the JST connectors)
All outputs generated
Other:
- company: Opulo -> Opulo.io
Changed lines of the file:
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@@
   (title_block
     (title "LumenPnP Motherboard")
-    (date "2022-09-09")
-    (rev "004A")
-    (company "Opulo")
+    (date "2022-10-06")
+    (rev "04A")
+    (company "Opulo.io")
     (comment 1 "Reengineered by Magpie")
   )
